Commit message: Update model_Robot.xacro

File: model_Robot.xacro (robot description, xacro)
@@ -170,5 +170,5 @@
       </geometry>
     </collision>
-    <xacro:inertial_box mass="0.8" x="0.18" y="0.028" z="0.085">
+    <xacro:inertial_box mass="2" x="0.18" y="0.028" z="0.085">
         <origin xyz="0 0 0" rpy="0 0 0"/>
     </xacro:inertial_box>
@@ -179,7 +179,7 @@
   <!-- Joint between link_0 and link_24 -->
   <joint name="joint_24" type="revolute">
-    <parent link="base_link"/>
+    <parent link="link_0"/>
     <child link="link_24"/>
-    <origin xyz="0.503 -0.166 0.079" rpy="0 0 0"/>
+    <origin xyz="0.257 -0.158 0.079"  rpy= "-6.845 0 0"/>
     <axis xyz="1 0 0"/>
     <limit effort="5.0" velocity="1.0" lower="-0.540" upper="0.540"/>
@@ -197,6 +197,6 @@
       </geometry>
     </collision>
-    <xacro:inertial_box mass="0.8" x="0.18" y="0.028" z="0.085">
-        <origin xyz="0 0 0" rpy="0 0 0"/>
+    <xacro:inertial_box mass="2" x="0.18" y="0.028" z="0.085">
+        <origin xyz="0 0 0" rpy= " 0 0 0"/>
     </xacro:inertial_box>
   </link>
@@ -206,7 +206,7 @@
    <!-- Joint between link_0 and link_25 -->
   <joint name="joint_25" type="revolute">
-    <parent link="base_link"/>
+    <parent link="link_0"/>
     <child link="link_25"/>
-    <origin xyz="0.503 0.166 0.079" rpy="0 0 0"/>
+    <origin xyz="0.257 0.1427 0.079" rpy="6.84 0 0"/>
     <axis xyz="1 0 0"/>
     <limit effort="5.0" velocity="1.0" lower="-0.540" upper="0.540"/>
@@ -235,5 +235,5 @@
     <parent link="link_24"/>
     <child link="link_27"/>
-    <origin xyz="0.681 -0.159 0.028" rpy="0 0 0"/>
+    <origin xyz="0.171 0.03 -0.001" rpy="0 0 0"/>
     <axis xyz="1 0 0"/>
    <limit lower="-0.2625" upper="0" effort="10.0" velocity="0.5"/>

Commit message: Update model_Robot.xacro

File: model_Robot.xacro (robot description, xacro)
@@ -181,5 +181,5 @@
     <parent link="link_0"/>
     <child link="link_24"/>
-    <origin xyz="0.257 -0.158 0.079"  rpy= "-6.845 0 0"/>
+    <origin xyz="0.257 -0.158 0.079"  rpy= "-5.77 0 0"/>
     <axis xyz="1 0 0"/>
     <limit effort="5.0" velocity="1.0" lower="-0.540" upper="0.540"/>
@@ -208,5 +208,5 @@
     <parent link="link_0"/>
     <child link="link_25"/>
-    <origin xyz="0.257 0.1427 0.079" rpy="6.84 0 0"/>
+    <origin xyz="0.257 0.1427 0.079" rpy="0 0 0"/>
     <axis xyz="1 0 0"/>
     <limit effort="5.0" velocity="1.0" lower="-0.540" upper="0.540"/>
@@ -235,5 +235,5 @@
     <parent link="link_24"/>
     <child link="link_27"/>
-    <origin xyz="0.171 0.03 -0.001" rpy="0 0 0"/>
+    <origin xyz="0.1806 0.023 -0.05" rpy="0 0 0"/>
     <axis xyz="1 0 0"/>
    <limit lower="-0.2625" upper="0" effort="10.0" velocity="0.5"/>
@@ -263,5 +263,5 @@
     <parent link="link_25"/>
     <child link="link_28"/>
-    <origin xyz="0.681 0.16 0.028" rpy="0 0 0"/>
+    <origin xyz="0.178 0 -0.05" rpy="0 0 0"/>
     <axis xyz="1 0 0"/>
    <limit lower="-0.2625" upper="0" effort="10.0" velocity="0.5"/>

Commit message: Update model_Robot.xacro

File: model_Robot.xacro (robot description, xacro)
@@ -2,18 +2,21 @@
 <robot xmlns:xacro="http://www.ros.org/wiki/xacro"  name="ROBOT_PROJECT_VERSION_02">
 <xacro:include filename="inertial_macros.xacro" />
-    <material name="white">
-        <color rgba="1 1 1 1" />
-    </material>
-    <material name="orange">
-        <color rgba="1 0.3 0.1 1"/>
-    </material>
-    <material name="blue">
-        <color rgba="0.2 0.2 1 1"/>
-    </material>
-    <material name="black">
-        <color rgba="0 0 0 1"/>
-    </material>
+   <material name="white">
+    <color rgba="1 1 1 1" />
+  </material>
+  <material name="orange">
+    <color rgba="1 0.3 0.1 1"/>
+  </material>
+  <material name="blue">
+    <color rgba="0.2 0.2 1 1"/>
+  </material>
+  <material name="black">
+    <color rgba="0 0 0 1"/>
+  </material>
  <material name="red">
-     <color rgba="1 0 0 1"/>
+    <color rgba="1 0 0 1"/>
+ </material>
+ <material name="grey">
+    <color rgba="0.5 0.5 0.5 1"/>
  </material>
 <!-- Link -->
@@ -33,10 +36,10 @@
     <visual>
       <geometry>
-        <mesh filename="/root/ROBOT_PROJECT_02_ws/BODY_PART_Version3.dae" scale="1 1 1"/>
-      </geometry>
-    </visual>
-    <collision>
-      <geometry>
-        <mesh filename="/root/ROBOT_PROJECT_02_ws/BODY_PART_Version3.dae" scale="1 1 1"/>
+        <mesh filename="file:///root/ROBOT_PROJECT_02_ws/BODY_PART_Version3.dae" scale="1 1 1"/>
+      </geometry>
+    </visual>
+    <collision>
+      <geometry>
+        <mesh filename="file:///root/ROBOT_PROJECT_02_ws/BODY_PART_Version3.dae" scale="1 1 1"/>
       </geometry>
     </collision>
@@ -46,5 +49,5 @@
   </link>
     <gazebo reference="link_0">
-    <material>Gazebo/White</material>
+    <material>Gazebo/Red</material>
     </gazebo>
 <!-- Joint between base_link and link_0  -->
@@ -58,18 +61,18 @@
     <visual>
       <geometry>
-        <mesh filename="/root/ROBOT_PROJECT_02_ws/Wheel_partV3.dae" scale="1 1 1"/>
-      </geometry>
-    </visual>
-    <collision>
-      <geometry>
-        <mesh filename="/root/ROBOT_PROJECT_02_ws/Wheel_partV3.dae" scale="1 1 1"/>
-      </geometry>
-    </collision>
-    <xacro:inertial_cylinder mass="4" length ="0.060" radius ="0.075" >
-        <origin xyz="0 0 0" rpy="0 0 0"/>
-    </xacro:inertial_cylinder>
-  </link>
-    <gazebo reference="link_0">
-    <material>Gazebo/White</material>
+        <mesh filename="file:///root/ROBOT_PROJECT_02_ws/Wheel_partV3.dae" scale="1 1 1"/>
+      </geometry>
+    </visual>
+    <collision>
+      <geometry>
+        <mesh filename="file:///root/ROBOT_PROJECT_02_ws/Wheel_partV3.dae" scale="1 1 1"/>
+      </geometry>
+    </collision>
+    <xacro:inertial_cylinder mass="4" length ="0.060" radius ="0.075" >
+        <origin xyz="0 0 0" rpy="0 0 0"/>
+    </xacro:inertial_cylinder>
+  </link>
+    <gazebo reference="link_0">
+    <material>Gazebo/Black</material>
     </gazebo>
   <!-- Joint between link_0 and link_14 -->
@@ -84,18 +87,18 @@
     <visual>
       <geometry>
-        <mesh filename="/root/ROBOT_PROJECT_02_ws/Wheel_partV3.dae" scale="1 1 1"/>
-      </geometry>
-    </visual>
-    <collision>
-      <geometry>
-        <mesh filename="/root/ROBOT_PROJECT_02_ws/Wheel_partV3.dae" scale="1 1 1"/>
-      </geometry>
-    </collision>
-    <xacro:inertial_cylinder mass="4" length ="0.060" radius ="0.075" >
-        <origin xyz="0 0 0" rpy="0 0 0"/>
-    </xacro:inertial_cylinder>
-  </link>
-    <gazebo reference="link_0">
-    <material>Gazebo/White</material>
+        <mesh filename="file:///root/ROBOT_PROJECT_02_ws/Wheel_partV3.dae" scale="1 1 1"/>
+      </geometry>
+    </visual>
+    <collision>
+      <geometry>
+        <mesh filename="file:///root/ROBOT_PROJECT_02_ws/Wheel_partV3.dae" scale="1 1 1"/>
+      </geometry>
+    </collision>
+    <xacro:inertial_cylinder mass="4" length ="0.060" radius ="0.075" >
+        <origin xyz="0 0 0" rpy="0 0 0"/>
+    </xacro:inertial_cylinder>
+  </link>
+    <gazebo reference="link_0">
+    <material>Gazebo/Black</material>
     </gazebo>
   <!-- Joint between link_0 and link_15 -->
@@ -110,18 +113,18 @@
     <visual>
       <geometry>
-        <mesh filename="/root/ROBOT_PROJECT_02_ws/Wheel_partV3.dae" scale="1 1 1"/>
-      </geometry>
-    </visual>
-    <collision>
-      <geometry>
-        <mesh filename="/root/ROBOT_PROJECT_02_ws/Wheel_partV3.dae" scale="1 1 1"/>
-      </geometry>
-    </collision>
-    <xacro:inertial_cylinder mass="4" length ="0.060" radius ="0.075" >
-        <origin xyz="0 0 0" rpy="0 0 0"/>
-    </xacro:inertial_cylinder>
-  </link>
-    <gazebo reference="link_0">
-    <material>Gazebo/White</material>
+        <mesh filename="file:///root/ROBOT_PROJECT_02_ws/Wheel_partV3.dae" scale="1 1 1"/>
+      </geometry>
+    </visual>
+    <collision>
+      <geometry>
+        <mesh filename="file:///root/ROBOT_PROJECT_02_ws/Wheel_partV3.dae" scale="1 1 1"/>
+      </geometry>
+    </collision>
+    <xacro:inertial_cylinder mass="4" length ="0.060" radius ="0.075" >
+        <origin xyz="0 0 0" rpy="0 0 0"/>
+    </xacro:inertial_cylinder>
+  </link>
+    <gazebo reference="link_0">
+    <material>Gazebo/Black</material>
     </gazebo>
   <!-- Joint between link_0 and link_16 -->
@@ -136,18 +139,18 @@
     <visual>
       <geometry>
-        <mesh filename="/root/ROBOT_PROJECT_02_ws/Wheel_partV3.dae" scale="1 1 1"/>
-      </geometry>
-    </visual>
-    <collision>
-      <geometry>
-        <mesh filename="/root/ROBOT_PROJECT_02_ws/Wheel_partV3.dae" scale="1 1 1"/>
-      </geometry>
-    </collision>
-    <xacro:inertial_cylinder mass="4" length ="0.060" radius ="0.075" >
-        <origin xyz="0 0 0" rpy="0 0 0"/>
-    </xacro:inertial_cylinder>
-  </link>
-    <gazebo reference="link_0">
-    <material>Gazebo/White</material>
+        <mesh filename="file:///root/ROBOT_PROJECT_02_ws/Wheel_partV3.dae" scale="1 1 1"/>
+      </geometry>
+    </visual>
+    <collision>
+      <geometry>
+        <mesh filename="file:///root/ROBOT_PROJECT_02_ws/Wheel_partV3.dae" scale="1 1 1"/>
+      </geometry>
+    </collision>
+    <xacro:inertial_cylinder mass="4" length ="0.060" radius ="0.075" >
+        <origin xyz="0 0 0" rpy="0 0 0"/>
+    </xacro:inertial_cylinder>
+  </link>
+    <gazebo reference="link_0">
+    <material>Gazebo/Black</material>
     </gazebo>
   <!-- Joint between link_0 and link_17 -->
@@ -162,10 +165,10 @@
     <visual>
       <geometry>
-        <mesh filename="/root/ROBOT_PROJECT_02_ws/LINK_V3.dae" scale="1 1 1"/>
-      </geometry>
-    </visual>
-    <collision>
-      <geometry>
-        <mesh filename="/root/ROBOT_PROJECT_02_ws/LINK_V3.dae" scale="1 1 1"/>
+        <mesh filename="file:///root/ROBOT_PROJECT_02_ws/LINK_V3.dae" scale="1 1 1"/>
+      </geometry>
+    </visual>
+    <collision>
+      <geometry>
+        <mesh filename="file:///root/ROBOT_PROJECT_02_ws/LINK_V3.dae" scale="1 1 1"/>
       </geometry>
     </collision>
@@ -181,6 +184,6 @@
     <parent link="link_0"/>
     <child link="link_24"/>
-    <origin xyz="0.257 -0.158 0.079"  rpy= "-5.77 0 0"/>
-    <axis xyz="1 0 0"/>
+    <origin xyz="0.257 -0.158 0.079"  rpy= "-6.3 0 0"/>
+    <axis xyz="0 1 0"/>
     <limit effort="5.0" velocity="1.0" lower="-0.540" upper="0.540"/>
   </joint>
@@ -189,10 +192,10 @@
     <visual>
       <geometry>
-        <mesh filename="/root/ROBOT_PROJECT_02_ws/LINK_V3.dae" scale="1 1 1"/>
-      </geometry>
-    </visual>
-    <collision>
-      <geometry>
-        <mesh filename="/root/ROBOT_PROJECT_02_ws/LINK_V3.dae" scale="1 1 1"/>
+        <mesh filename="file:///root/ROBOT_PROJECT_02_ws/LINK_V3.dae" scale="1 1 1"/>
+      </geometry>
+    </visual>
+    <collision>
+      <geometry>
+        <mesh filename="file:///root/ROBOT_PROJECT_02_ws/LINK_V3.dae" scale="1 1 1"/>
       </geometry>
     </collision>
@@ -209,5 +212,5 @@
     <child link="link_25"/>
     <origin xyz="0.257 0.1427 0.079" rpy="0 0 0"/>
-    <axis xyz="1 0 0"/>
+    <axis xyz="0 1 0"/>
     <limit effort="5.0" velocity="1.0" lower="-0.540" upper="0.540"/>
   </joint>
@@ -216,10 +219,10 @@
     <visual>
       <geometry>
-        <mesh filename="/root/ROBOT_PROJECT_02_ws/HAND1_V3dae.dae" scale="1 1 1"/>
-      </geometry>
-    </visual>
-    <collision>
-      <geometry>
-        <mesh filename="/root/ROBOT_PROJECT_02_ws/HAND1_V3dae.dae" scale="1 1 1"/>
+        <mesh filename="file:///root/ROBOT_PROJECT_02_ws/HAND1_V3dae.dae" scale="1 1 1"/>
+      </geometry>
+    </visual>
+    <collision>
+      <geometry>
+        <mesh filename="file:///root/ROBOT_PROJECT_02_ws/HAND1_V3dae.dae" scale="1 1 1"/>
       </geometry>
     </collision>
@@ -229,5 +232,5 @@
   </link>
     <gazebo reference="link_0">
-    <material>Gazebo/White</material>
+    <material>Gazebo/Grey</material>
     </gazebo>
   <!-- Joint between link_24 and link_27 -->
@@ -236,6 +239,6 @@
     <child link="link_27"/>
     <origin xyz="0.1806 0.023 -0.05" rpy="0 0 0"/>
-    <axis xyz="1 0 0"/>
-   <limit lower="-0.2625" upper="0" effort="10.0" velocity="0.5"/>
+    <axis xyz="0 1 0"/>
+   <limit lower="-0.02" upper="0.02" effort="10.0" velocity="0.5"/>
    <dynamics damping="0.1" friction="0.05"/>
   </joint>
@@ -244,10 +247,10 @@
     <visual>
       <geometry>
-        <mesh filename="/root/ROBOT_PROJECT_02_ws/HAND2_V3dae.dae" scale="1 1 1"/>
-      </geometry>
-    </visual>
-    <collision>
-      <geometry>
-        <mesh filename="/root/ROBOT_PROJECT_02_ws/HAND2_V3dae.dae" scale="1 1 1"/>
+        <mesh filename="file:///root/ROBOT_PROJECT_02_ws/HAND2_V3dae.dae" scale="1 1 1"/>
+      </geometry>
+    </visual>
+    <collision>
+      <geometry>
+        <mesh filename="file:///root/ROBOT_PROJECT_02_ws/HAND2_V3dae.dae" scale="1 1 1"/>
       </geometry>
     </collision>
@@ -257,5 +260,5 @@
   </link>
     <gazebo reference="link_0">
-    <material>Gazebo/White</material>
+    <material>Gazebo/Grey</material>
     </gazebo>
   <!-- Joint between link_25 and link_28 -->
@@ -264,5 +267,5 @@
     <child link="link_28"/>
     <origin xyz="0.178 0 -0.05" rpy="0 0 0"/>
-    <axis xyz="1 0 0"/>
+    <axis xyz="0 1 0"/>
    <limit lower="-0.2625" upper="0" effort="10.0" velocity="0.5"/>
    <dynamics damping="0.1" friction="0.05"/>

Commit message: Update model_Robot.xacro

File: model_Robot.xacro (robot description, xacro)
@@ -107,5 +107,5 @@
     <child link="link_15"/>
     <origin xyz="-0.130194 -0.211467 0.0" rpy="0 0 0"/>
-    <axis xyz="0 1 0"/>
+    <axis xyz="0 -1 0"/>
   </joint>
     <!-- Link 16(RIGHT_FRONT PART) -->
@@ -133,5 +133,5 @@
     <child link="link_16"/>
     <origin xyz="0.080 -0.211467 0.0" rpy="0 0 0"/>
-    <axis xyz="0 1 0"/>
+    <axis xyz="0 -1 0"/>
   </joint>
       <!-- Link 17(LEFT_FRONT PART) -->
@@ -185,6 +185,6 @@
     <child link="link_24"/>
     <origin xyz="0.257 -0.158 0.079"  rpy= "-6.3 0 0"/>
-    <axis xyz="0 1 0"/>
-    <limit effort="5.0" velocity="1.0" lower="-0.540" upper="0.540"/>
+    <axis xyz="0 -1 0"/>
+    <limit effort="5.0" velocity="1.0" lower="-0.10" upper="2.50"/>
   </joint>
      <!--  Link 25 (ARM LEFT)-->
@@ -212,6 +212,6 @@
     <child link="link_25"/>
     <origin xyz="0.257 0.1427 0.079" rpy="0 0 0"/>
-    <axis xyz="0 1 0"/>
-    <limit effort="5.0" velocity="1.0" lower="-0.540" upper="0.540"/>
+    <axis xyz="0 -1 0"/>
+    <limit effort="5.0" velocity="1.0" lower="-0.10" upper="2.50"/>
   </joint>
   <!-- Link 27 (Hydraulic right)-->
@@ -240,5 +240,5 @@
     <origin xyz="0.1806 0.023 -0.05" rpy="0 0 0"/>
     <axis xyz="0 1 0"/>
-   <limit lower="-0.02" upper="0.02" effort="10.0" velocity="0.5"/>
+   <limit lower="-0.01" upper="0.055" effort="10.0" velocity="0.5"/>
    <dynamics damping="0.1" friction="0.05"/>
   </joint>
@@ -267,6 +267,6 @@
     <child link="link_28"/>
     <origin xyz="0.178 0 -0.05" rpy="0 0 0"/>
-    <axis xyz="0 1 0"/>
-   <limit lower="-0.2625" upper="0" effort="10.0" velocity="0.5"/>
+    <axis xyz="0 -1 0"/>
+   <limit lower="-0.01" upper="0.055" effort="10.0" velocity="0.5"/>
    <dynamics damping="0.1" friction="0.05"/>
   </joint>

Commit message: Update model_Robot.xacro

File: model_Robot.xacro (robot description, xacro)
@@ -44,5 +44,5 @@
       </geometry>
     </collision>
-    <xacro:inertial_box mass="6" x="0.480" y="0.500" z="0.">
+    <xacro:inertial_box mass="10" x="0.480" y="0.500" z="0.">
         <origin xyz="0 0 0" rpy="0 0 0"/>
     </xacro:inertial_box>
@@ -69,5 +69,5 @@
       </geometry>
     </collision>
-    <xacro:inertial_cylinder mass="4" length ="0.060" radius ="0.075" >
+    <xacro:inertial_cylinder mass="2" length ="0.060" radius ="0.075" >
         <origin xyz="0 0 0" rpy="0 0 0"/>
     </xacro:inertial_cylinder>
@@ -95,5 +95,5 @@
       </geometry>
     </collision>
-    <xacro:inertial_cylinder mass="4" length ="0.060" radius ="0.075" >
+    <xacro:inertial_cylinder mass="2" length ="0.060" radius ="0.075" >
         <origin xyz="0 0 0" rpy="0 0 0"/>
     </xacro:inertial_cylinder>
@@ -121,5 +121,5 @@
       </geometry>
     </collision>
-    <xacro:inertial_cylinder mass="4" length ="0.060" radius ="0.075" >
+    <xacro:inertial_cylinder mass="2" length ="0.060" radius ="0.075" >
         <origin xyz="0 0 0" rpy="0 0 0"/>
     </xacro:inertial_cylinder>
@@ -147,5 +147,5 @@
       </geometry>
     </collision>
-    <xacro:inertial_cylinder mass="4" length ="0.060" radius ="0.075" >
+    <xacro:inertial_cylinder mass="2" length ="0.060" radius ="0.075" >
         <origin xyz="0 0 0" rpy="0 0 0"/>
     </xacro:inertial_cylinder>
@@ -173,5 +173,5 @@
       </geometry>
     </collision>
-    <xacro:inertial_box mass="2" x="0.18" y="0.028" z="0.085">
+    <xacro:inertial_box mass="0.2" x="0.18" y="0.028" z="0.085">
         <origin xyz="0 0 0" rpy="0 0 0"/>
     </xacro:inertial_box>
@@ -184,5 +184,5 @@
     <parent link="link_0"/>
     <child link="link_24"/>
-    <origin xyz="0.257 -0.158 0.079"  rpy= "-6.3 0 0"/>
+    <origin xyz="0.257 -0.158 0.079"  rpy= "-6.3 0.05 0"/>
     <axis xyz="0 -1 0"/>
     <limit effort="5.0" velocity="1.0" lower="-0.10" upper="2.50"/>
@@ -200,5 +200,5 @@
       </geometry>
     </collision>
-    <xacro:inertial_box mass="2" x="0.18" y="0.028" z="0.085">
+    <xacro:inertial_box mass="0.2" x="0.18" y="0.028" z="0.085">
         <origin xyz="0 0 0" rpy= " 0 0 0"/>
     </xacro:inertial_box>
@@ -211,5 +211,5 @@
     <parent link="link_0"/>
     <child link="link_25"/>
-    <origin xyz="0.257 0.1427 0.079" rpy="0 0 0"/>
+    <origin xyz="0.257 0.1427 0.079" rpy="0 0.05 0"/>
     <axis xyz="0 -1 0"/>
     <limit effort="5.0" velocity="1.0" lower="-0.10" upper="2.50"/>
@@ -227,5 +227,5 @@
       </geometry>
     </collision>
-    <xacro:inertial_box mass="0.2" x="0.15" y="0.090" z="0.15">
+    <xacro:inertial_box mass="0.1" x="0.10" y="0.060" z="0.10">
         <origin xyz="0 0 0" rpy="0 0 0"/>
     </xacro:inertial_box>
@@ -255,5 +255,5 @@
       </geometry>
     </collision>
-    <xacro:inertial_box mass="0.2" x="0.15" y="0.090" z="0.15">
+    <xacro:inertial_box mass="0.1" x="0.10" y="0.060" z="0.10">
         <origin xyz="0 0 0" rpy="0 0 0"/>
     </xacro:inertial_box>
