Commit message: Update model_Robot_version02.xacro

File: model_Robot_version02.xacro (robot description, xacro)
@@ -38,4 +38,5 @@
         <mesh filename="file:///root/ROBOT_PROJECT_02_ws/BODY_PART_Version3.dae" scale="1 1 1"/>
       </geometry>
+      <material name="red"/>
     </visual>
     <collision>
@@ -63,8 +64,9 @@
         <cylinder length="0.06" radius="0.072" />
       </geometry>
-    </visual>
-    <collision>
-      <geometry>
-        <cylinder length="0.06" radius="0.072" />
+      <material name="black"/>
+    </visual>
+    <collision>
+      <geometry>
+       <cylinder length="0.06" radius="0.072" />
       </geometry>
     </collision>
@@ -89,4 +91,5 @@
         <cylinder length="0.06" radius="0.072" />
       </geometry>
+      <material name="black"/>
     </visual>
     <collision>
@@ -115,4 +118,5 @@
         <cylinder length="0.06" radius="0.072" />
       </geometry>
+      <material name="black"/>
     </visual>
     <collision>
@@ -141,4 +145,5 @@
         <cylinder length="0.06" radius="0.072" />
       </geometry>
+      <material name="black"/>
     </visual>
     <collision>
@@ -159,5 +164,5 @@
     <child link="link_17"/>
     <origin xyz="0.080 0.208533 0.0" rpy="1.57 0 0"/>
-    <axis xyz="0 0 1"/>
+    <axis xyz="0 0 -1"/>
   </joint>
    <!--  Link 24 (ARM RIGHT)-->
@@ -167,4 +172,5 @@
         <mesh filename="file:///root/ROBOT_PROJECT_02_ws/LINK_V3.dae" scale="1 1 1"/>
       </geometry>
+      <material name="white"/>
     </visual>
     <collision>
@@ -193,4 +199,5 @@
         <mesh filename="file:///root/ROBOT_PROJECT_02_ws/LINK_V3.dae" scale="1 1 1"/>
       </geometry>
+      <material name="white"/>
     </visual>
     <collision>
@@ -219,4 +226,5 @@
         <mesh filename="file:///root/ROBOT_PROJECT_02_ws/HAND1_V3dae.dae" scale="1 1 1"/>
       </geometry>
+      <material name="grey"/>
     </visual>
     <collision>
@@ -246,4 +254,5 @@
         <mesh filename="file:///root/ROBOT_PROJECT_02_ws/HAND2_V3dae.dae" scale="1 1 1"/>
       </geometry>
+      <material name="grey"/>
     </visual>
     <collision>
